File: HierSheets/line.kicad_sch (KiCad schematic)
At the start: 0 parts

Commit message: Added line sensor
Parts:
- added C10, C11, C12, C9: C0.1uF, symbol Device:C
- added D10, D11, D12, D17, D18, D19, D20, D21, D22, D23, D24, D25, D26, D27, D28, D9: SFH_4656-Z, symbol Device:LED
- added Q10, Q11, Q12, Q17, Q18, Q19, Q20, Q21, Q22, Q23, Q24, Q25, Q26, Q27, Q28, Q9: SFH309, LED_THT:LED_D3.0mm_Clear, symbol Sensor_Optical:SFH309
- added R38, R39, R40, R41, R54, R55, R56, R57, R62, R63, R64, R65, R70, R71, R72, R73: 750R, symbol Device:R
- added R42, R43, R44, R45, R58, R59, R60, R61, R66, R67, R68, R69, R74, R75, R76, R77: 10kR, symbol Device:R
- added U13, U14, U15, U16: ADS1115IDGS, Package_SO:TSSOP-10_3x3mm_P0.5mm, symbol Analog_ADC:ADS1115IDGS
Connections:
- new net: D25.1 (K), R70.2
- new net: Q10.2 (E), R43.1, U14.5 (AIN1)
- new net: D19.1 (K), R56.2
- new net: Q20.2 (E), R61.1, U13.7 (AIN3)
- new net: D22.1 (K), R63.2
- new net: Q22.2 (E), R67.1, U16.5 (AIN1)
- new net: Q9.2 (E), R42.1, U14.4 (AIN0)
- new net: D21.1 (K), R62.2
- new net: D20.1 (K), R57.2
- new net: D24.1 (K), R65.2
- new net: D18.1 (K), R55.2
- new net: Q12.2 (E), R45.1, U14.7 (AIN3)
- new net: Q28.2 (E), R77.1, U15.7 (AIN3)
- new net: D11.1 (K), R40.2
- new net: Q26.2 (E), R75.1, U15.5 (AIN1)
- new net: D17.1 (K), R54.2
- new net: Q18.2 (E), R59.1, U13.5 (AIN1)
- new net: Q21.2 (E), R66.1, U16.4 (AIN0)
- new net: Q23.2 (E), R68.1, U16.6 (AIN2)
- new net: Q25.2 (E), R74.1, U15.4 (AIN0)
- new net: D9.1 (K), R38.2
- new net: Q27.2 (E), R76.1, U15.6 (AIN2)
- new net: Q17.2 (E), R58.1, U13.4 (AIN0)
- new net: D27.1 (K), R72.2
- new net: Q24.2 (E), R69.1, U16.7 (AIN3)
- new net: D10.1 (K), R39.2
- new net: D23.1 (K), R64.2
- new net: Q19.2 (E), R60.1, U13.6 (AIN2)
- new net: D12.1 (K), R41.2
- new net: D28.1 (K), R73.2
- new net: D26.1 (K), R71.2
- new net: Q11.2 (E), R44.1, U14.6 (AIN2)
- new net 3V3: C10.1, C11.1, C12.1, C9.1, Q10.1 (C), Q11.1 (C), Q12.1 (C), Q17.1 (C), Q18.1 (C), Q19.1 (C), Q20.1 (C), Q21.1 (C), Q22.1 (C), Q23.1 (C), Q24.1 (C), Q25.1 (C), Q26.1 (C), Q27.1 (C), Q28.1 (C), Q9.1 (C), R38.1, R39.1, R40.1, R41.1, R54.1, R55.1, R56.1, R57.1, R62.1, R63.1, R64.1, R65.1, R70.1, R71.1, R72.1, R73.1, U13.8 (VDD), U14.1 (ADDR), U14.8 (VDD), U15.8 (VDD), U16.8 (VDD)
- new net GNDD: C10.2, C11.2, C12.2, C9.2, D10.2 (A), D11.2 (A), D12.2 (A), D17.2 (A), D18.2 (A), D19.2 (A), D20.2 (A), D21.2 (A), D22.2 (A), D23.2 (A), D24.2 (A), D25.2 (A), D26.2 (A), D27.2 (A), D28.2 (A), D9.2 (A), R42.2, R43.2, R44.2, R45.2, R58.2, R59.2, R60.2, R61.2, R66.2, R67.2, R68.2, R69.2, R74.2, R75.2, R76.2, R77.2, U13.1 (ADDR), U13.3 (GND), U14.3 (GND), U15.3 (GND), U16.3 (GND)
- new net I2C.SCL: U13.10 (SCL), U14.10 (SCL), U15.1 (ADDR), U15.10 (SCL), U16.10 (SCL)
- new net I2C.SDA: U13.9 (SDA), U14.9 (SDA), U15.9 (SDA), U16.1 (ADDR), U16.9 (SDA)
