File: HierSheets/MotorDriver.kicad_sch (KiCad schematic)
At the start: 44 parts, among them U10 INA240A1D, U11 INA240A1D, U12 INA240A1D, U2 74LVC1G04, U3 74LVC1G04, U4 74LVC1G04, U5 74LVC1G04, U6 TB6612FNG, U7 TB6612FNG, U8 PCF8574TS, U9 INA240A1D

Commit message: .
Connections:
- net MotorDrawAnalogValue1 renamed DrawAnalog1
- net MotorDrawAnalogValue2 renamed DrawAnalog2
- net MotorDrawAnalogValue3 renamed DrawAnalog3
- net MotorDrawAnalogValue4 renamed DrawAnalog4
Changed lines of the file:
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@@
 	(wire
 		(pts
-			(xy 133.35 102.87) (xy 142.24 102.87)
+			(xy 134.62 102.87) (xy 142.24 102.87)
 		)
 		(stroke
@@
 	(wire
 		(pts
-			(xy 133.35 163.83) (xy 142.24 163.83)
+			(xy 134.62 163.83) (xy 142.24 163.83)
 		)
 		(stroke
@@
 	(wire
 		(pts
-			(xy 133.35 105.41) (xy 142.24 105.41)
+			(xy 134.62 105.41) (xy 142.24 105.41)
 		)
 		(stroke
@@
 	(wire
 		(pts
-			(xy 133.35 143.51) (xy 142.24 143.51)
+			(xy 134.62 143.51) (xy 142.24 143.51)
 		)
 		(stroke
@@
 	(wire
 		(pts
-			(xy 133.35 123.19) (xy 142.24 123.19)
+			(xy 134.62 123.19) (xy 142.24 123.19)
 		)
 		(stroke
@@
 	(wire
 		(pts
-			(xy 133.35 125.73) (xy 142.24 125.73)
+			(xy 134.62 125.73) (xy 142.24 125.73)
 		)
 		(stroke
@@
 	(wire
 		(pts
-			(xy 133.35 146.05) (xy 142.24 146.05)
+			(xy 134.62 146.05) (xy 142.24 146.05)
 		)
 		(stroke
@@
 	(wire
 		(pts
-			(xy 133.35 166.37) (xy 142.24 166.37)
+			(xy 134.62 166.37) (xy 142.24 166.37)
 		)
 		(stroke
@@
 	)
 	(label "ENC3B"
-		(at 133.35 146.05 180)
+		(at 134.62 146.05 180)
 		(effects
 			(font
@@
 	)
 	(label "ENC1B"
-		(at 133.35 105.41 180)
+		(at 134.62 105.41 180)
 		(effects
 			(font
@@
 	)
 	(label "ENC2B"
-		(at 133.35 125.73 180)
+		(at 134.62 125.73 180)
 		(effects
 			(font
@@
 	)
 	(label "ENC4B"
-		(at 133.35 166.37 180)
+		(at 134.62 166.37 180)
 		(effects
 			(font
@@
 	)
 	(label "ENC3A"
-		(at 133.35 143.51 180)
+		(at 134.62 143.51 180)
 		(effects
 			(font
@@
 	)
 	(label "ENC1A"
-		(at 133.35 102.87 180)
+		(at 134.62 102.87 180)
 		(effects
 			(font
@@
 	)
 	(label "ENC2A"
-		(at 133.35 123.19 180)
+		(at 134.62 123.19 180)
 		(effects
 			(font
@@
 	)
 	(label "ENC4A"
-		(at 133.35 163.83 180)
+		(at 134.62 163.83 180)
 		(effects
 			(font
@@
 		)
 	)
-	(hierarchical_label "MotorDrawAnalogValue1"
+	(hierarchical_label "DrawAnalog1"
 		(shape output)
 		(at 205.74 95.25 0)
@@
 		)
 	)
-	(hierarchical_label "MotorDrawAnalogValue4"
+	(hierarchical_label "DrawAnalog4"
 		(shape output)
 		(at 205.74 102.87 0)
@@
 		)
 	)
-	(hierarchical_label "MotorDrawAnalogValue2"
+	(hierarchical_label "DrawAnalog2"
 		(shape output)
 		(at 205.74 97.79 0)
@@
 		)
 	)
-	(hierarchical_label "MotorDrawAnalogValue3"
+	(hierarchical_label "DrawAnalog3"
 		(shape output)
 		(at 205.74 100.33 0)

Commit message: Added kicker, interrupt, I2C pullups, buck converter, button
Parts:
- renumbered C1 to C2, C2 to C3, C3 to C4, C4 to C5, C5 to C6, C6 to C7, C7 to C8, C8 to C9, R4 to R10, R5 to R11, R6 to R12, R7 to R13, R8 to R14, R9 to R15, R10 to R16, R11 to R17, R12 to R18, R13 to R19, R14 to R20, R15 to R21, R16 to R22, R17 to R23, R1 to R3, R18 to R4, R19 to R5, R20 to R6, R21 to R7, R2 to R8, R3 to R9, U9 to U10, U10 to U11, U11 to U12, U12 to U13, U2 to U3, U3 to U4, U4 to U5, U5 to U6, U6 to U7, U7 to U8, U8 to U9
Connections:
- net GNDD: now also U9.6 (A0), U9.7 (A1), U9.9 (A2)
- net H_INTN: now reaches U9.1 (~{INT})
Other:
- note added: "0x20 - 0x27"
- note added: "0x40"
- note added: "0x41"
