File: Prototyp_0.1.kicad_sch (KiCad schematic)
At the start: 4 parts, among them U1 ESP32-S3-WROOM-1U

Commit message: .
Connections:
- net DribblerDriver/DIR: no longer U1.24 (IO47)
- net DribblerDriver/PWM: no longer U1.25 (IO48)
- net KickerDriver/DIR: no longer U1.22 (IO14)
- net KickerDriver/PWM: no longer U1.21 (IO13)
Other:
- added sheet StatusLEDs (HierSheets/statusdis.kicad_sch)
- sheet BuckConverter ports: added IN12V, OUT5V; removed 12V, 5V
- sheet DriversSupply ports: added IN, OUT, Status; removed INPUT, OUTPUT, RandomAhhData
- sheet MotorDriver ports: added DrawAnalog1, DrawAnalog2, DrawAnalog3, DrawAnalog4; removed MotorDrawAnalogValue1, MotorDrawAnalogValue2, MotorDrawAnalogValue3, MotorDrawAnalogValue4
- note removed: "CONTROL"
- note removed: "DRIVERS"
- note removed: "SENSORS"
- note removed: "STATUS"
