File: Prototyp_0.1.kicad_pcb (KiCad board)
At the start: 2 copper layers, 158 x 115.5 mm, 25 parts, among them U1 ESP32-S3-WROOM-1U, U10 INA240A1D, U11 INA240A1D, U12 INA240A1D, U2 74LVC1G04, U3 74LVC1G04, U4 74LVC1G04, U5 74LVC1G04, U6 TB6612FNG, U7 TB6612FNG, U8 PCF8574TS, U9 INA240A1D

Commit message: Added Libs folder and lib for eFuse
Parts:
- added REF**: VQFN24_RGE_TEX, TPS25983:VQFN24_RGE_TEX, F.Cu at (160.5, 38.0)

Commit message: Added kicker, interrupt, I2C pullups, buck converter, button
Parts:
- added AI_port(Raspberry)1: USB_C_Plug_USB2.0, Connector_USB:USB_C_Plug_Molex_105444, F.Cu at (186.3, 20.5)
- added D5: 1.5SMCxxCA, Diode_SMD:D_SMC, F.Cu at (187.0, 28.9)
- added D6: SS34, Diode_SMD:D_SMA, F.Cu at (204.7, 32.3)
- added LiDAR_port1: Conn_01x05, Connector_JST:JST_XH_B5B-XH-A_1x05_P2.50mm_Vertical, F.Cu at (185.0, 14.1)
- added Q1: IRLB8721PBF, Package_TO_SOT_THT:TO-220-3_Vertical, F.Cu at (203.8, 28.0)
- added Q2: SFH309, LED_THT:LED_D3.0mm_Clear, F.Cu at (202.3, 4.74)
- added Q3: SFH309, LED_THT:LED_D3.0mm_Clear, F.Cu at (202.3, 10.2)
- added Q4: SFH309, LED_THT:LED_D3.0mm_Clear, F.Cu at (208.2, 4.74)
- added Q5: SFH309, LED_THT:LED_D3.0mm_Clear, F.Cu at (208.2, 10.2)
- added Q6: SFH309, LED_THT:LED_D3.0mm_Clear, F.Cu at (214.0, 4.74)
- added Q7: SFH309, LED_THT:LED_D3.0mm_Clear, F.Cu at (214.0, 10.2)
- added Q8: SFH309, LED_THT:LED_D3.0mm_Clear, F.Cu at (219.9, 4.74)
- added Q9: SFH309, LED_THT:LED_D3.0mm_Clear, F.Cu at (219.9, 10.2)
- added RaspberryPower1: USB_A, Connector_USB:USB_A_Molex_105057_Vertical, F.Cu at (186.5, 8.76)
- added U1: XC6220B331MR, Package_TO_SOT_SMD:SOT-23-5, F.Cu at (216.7, 35.2)
- added U14: ADS1115IDGS, Package_SO:TSSOP-10_3x3mm_P0.5mm, F.Cu at (204.2, 15.2)
- added U15: ADS1115IDGS, Package_SO:TSSOP-10_3x3mm_P0.5mm, F.Cu at (204.2, 19.8)
- added U17: TPS25983, TPS25983:VQFN24_RGE_TEX, F.Cu at (217.3, 27.4)
- renumbered C1 to C2, C2 to C3, C5 to C6, C6 to C7, U9 to U10, U10 to U11, U11 to U12, U12 to U13, U1 to U2, U2 to U3, U3 to U4, U4 to U5, U5 to U6, U6 to U7, U7 to U8, U8 to U9
Connections:
- net /KickerDriver/DIR renamed /H_INTN
- net /KickerDriver/PWM renamed /KICKER
- net /MotorDriver/MotorDrawAnalogValue1 renamed /MDA1
- net /MotorDriver/MotorDrawAnalogValue2 renamed /MDA2
- net /MotorDriver/MotorDrawAnalogValue3 renamed /MDA3
- net /MotorDriver/MotorDrawAnalogValue4 renamed /MDA4
- BATTERY1 pad 1: GNDPWR -> Net-(BATTERY1-Pin_1)
- BATTERY1 pad 2: 12V -> 5V
- C6 pad 1: 12V -> 5V
- C7 pad 1: 12V -> 5V
- U2 pad 13: unconnected-(U1-USB_D--Pad13) -> /Ports/RPI_D-
- U2 pad 14: unconnected-(U1-USB_D+-Pad14) -> /Ports/RPI_D+
- U2 pad 23: unconnected-(U1-IO21-Pad23) -> /Ports/SupT_gpio
- U2 pad 24: /DribblerDriver/DIR -> unconnected-(U2-IO47-Pad24)
- U2 pad 25: /DribblerDriver/PWM -> unconnected-(U2-IO48-Pad25)
- U2 pad 36: unconnected-(U1-RXD0-Pad36) -> /Ports/LiDAR_TX
- U2 pad 37: unconnected-(U1-TXD0-Pad37) -> /Ports/LiDAR_RX
- U7 pad 13: 12V -> 5V
- U7 pad 14: 12V -> 5V
- U7 pad 24: 12V -> 5V
- U8 pad 13: 12V -> 5V
- U8 pad 14: 12V -> 5V
- U8 pad 24: 12V -> 5V
- U9 pad 1: unconnected-(U8-~{INT}-Pad1) -> /MotorDriver/H_INTN
- U9 pad 6: unconnected-(U8-A0-Pad6) -> GNDD
- U9 pad 7: unconnected-(U8-A1-Pad7) -> GNDD
- U9 pad 9: unconnected-(U8-A2-Pad9) -> GNDD
